File: Kicad_workshop_volundr_clock/Kicad_workshop_volundr_clock.kicad_pcb (KiCad board)
At the start: 2 copper layers, 1 part, among them U1 ESP-12F

Commit message: Update to work on Kicad 6.01
Other:
- net class Default removed
